File: Proton-KiCAD/DebugProbe.kicad_sch (KiCad schematic)
At the start: 52 parts, among them J3 DebugnBoot, U10 USBLC6-2P6

Commit message: Added Buttons and IMU
Parts:
- gave numbers to parts that had none: 50

Commit message: Fixed to higherarchical labels
Parts:
- removed C26: 10u, Capacitor_SMD:C_0805_2012Metric, symbol Device:C
- removed C27: 10u, Capacitor_SMD:C_0603_1608Metric, symbol Device:C
- removed CR2: BAT60JFILM, BAT60JFILM:CR_60JFILM_STM, symbol BAT60JFILM:BAT60JFILM
- removed J5: USB_C_Receptacle_USB2.0_14P, Connector_USB:USB_C_Receptacle_G-Switch_GT-USB-7010ASV, symbol Connector:USB_C_Receptacle_USB2.0_14P
- removed R18, R19: 5.1k, Resistor_SMD:R_0402_1005Metric, symbol Device:R_US
- removed U10: USBLC6-2P6, Package_TO_SOT_SMD:SOT-666, symbol Power_Protection:USBLC6-2P6
- removed U5: AP2112K-3.3, Package_TO_SOT_SMD:SOT-23-5, symbol Regulator_Linear:AP2112K-3.3
Connections:
- net +P3V3 renamed +3V3
- net PGND renamed GND
Other:
- note removed: "ESD Protection"
- note removed: "Power"
- moved on the sheet: C28, C30, C31, C32, C33, C34, C35, C36, C37, C38, C39, C40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
