File: Proton-KiCAD/Proton.kicad_pcb (KiCad board)
At the start: 4 copper layers, 20.3 x 99.1 mm, 119 parts, among them J1 USB_C_Receptacle_USB2.0_14P, J2 Conn_01x28_Pin, J3 DebugnBoot, J4 Conn_01x28_Pin, J5 USB_C_Receptacle_USB2.0_14P, J6 Conn_02x03_Top_Bottom, J7 UART-PINS, SW1 BOOTSEL, SW2 RESET, SW3 LEFT, SW4 RIGHT, U1 W25Q128JVS, U10 USBLC6-2P6, U2 NCP1117-3.3_SOT223, U3 RP2350_80QFN, U4 W25Q16JVUXIQ TR, U5 AP2112K-3.3, U6 RP2040, U7 SN74AUP1T17DCKR, U8 SN74AUP1T17DCKR, U9 USBLC6-2P6, Y1 ABM8-272-T3, Y2 ABM8-272-T3

Commit message: continued layout
Parts:
- removed C26: 10u, Capacitor_SMD:C_0805_2012Metric
- removed C27: 10u, Capacitor_SMD:C_0603_1608Metric
- removed CR2: BAT60JFILM, BAT60JFILM:CR_60JFILM_STM
- removed J2, J4: Conn_01x28_Pin, Connector_PinHeader_2.54mm:PinHeader_1x28_P2.54mm_Vertical
- removed R10, R9: 27, Resistor_SMD:R_0402_1005Metric
- removed R11: 3k, Resistor_SMD:R_0402_1005Metric
- removed R13: 2k, Resistor_SMD:R_0402_1005Metric
- removed R15: 1k, Resistor_SMD:R_0402_1005Metric
- removed R16: 510, Resistor_SMD:R_0402_1005Metric
- removed U10: USBLC6-2P6, Package_TO_SOT_SMD:SOT-666
- removed U5: AP2112K-3.3, Package_TO_SOT_SMD:SOT-23-5
- removed UD1: RED, LED_SMD:LED_0805_2012Metric
- removed UD2: YELLOW, LED_SMD:LED_0805_2012Metric
- removed UD3: GREEN, LED_SMD:LED_0805_2012Metric
- removed UD4: BLUE, LED_SMD:LED_0805_2012Metric
- added C43: 100n, Capacitor_SMD:C_0402_1005Metric, F.Cu at (79.3, 75.5)
- added C44: 100n, Capacitor_SMD:C_0402_1005Metric, F.Cu at (79.3, 77.5)
- added C45: 100n, Capacitor_SMD:C_0402_1005Metric, F.Cu at (79.3, 79.5)
- added C46: 100n, Capacitor_SMD:C_0402_1005Metric, F.Cu at (79.3, 81.4)
- added C47: 100n, Capacitor_SMD:C_0402_1005Metric, F.Cu at (82.1, 75.5)
- added C48: 100n, Capacitor_SMD:C_0402_1005Metric, F.Cu at (82.1, 77.5)
- added C49: 100n, Capacitor_SMD:C_0402_1005Metric, F.Cu at (82.1, 79.5)
- added C50: 100n, Capacitor_SMD:C_0402_1005Metric, F.Cu at (82.1, 81.4)
- added C51: 0.1u, Capacitor_SMD:C_0402_1005Metric, F.Cu at (85.0, 75.5)
- added C52: 2.2n, Capacitor_SMD:C_0402_1005Metric, F.Cu at (85.0, 77.5)
- added C53: 0.1u, Capacitor_SMD:C_0402_1005Metric, F.Cu at (85.0, 79.5)
- added C54: 0.1u, Capacitor_SMD:C_0402_1005Metric, F.Cu at (85.0, 81.4)
- added C55: 0.1u, Capacitor_SMD:C_0402_1005Metric, F.Cu at (87.9, 75.5)
- added C56: 4.7u, Capacitor_SMD:C_0402_1005Metric, F.Cu at (87.9, 77.5)
- added C57: 100n, Capacitor_SMD:C_0402_1005Metric, F.Cu at (87.9, 79.5)
- added C58: 100n, Capacitor_SMD:C_0402_1005Metric, F.Cu at (87.9, 81.4)
- added J8: HDMI_A, Connector_Video:HDMI_A_Molex_208658-1001_Horizontal, F.Cu at (143.5, 43.3)
- added R36: 1k, Resistor_SMD:R_0402_1005Metric, F.Cu at (79.3, 65.6)
- added R37: 10k, Resistor_SMD:R_0402_1005Metric, F.Cu at (79.3, 67.6)
- added R38: 1k, Resistor_SMD:R_0402_1005Metric, F.Cu at (79.3, 69.6)
- added R39: 10k, Resistor_SMD:R_0402_1005Metric, F.Cu at (79.3, 71.6)
- added R40: 1k, Resistor_SMD:R_0402_1005Metric, F.Cu at (79.3, 73.5)
- added R41: 10k, Resistor_SMD:R_0402_1005Metric, F.Cu at (82.2, 61.6)
- added R42: 1k, Resistor_SMD:R_0402_1005Metric, F.Cu at (82.2, 63.6)
- added R43: 10k, Resistor_SMD:R_0402_1005Metric, F.Cu at (82.2, 65.6)
- added R44: 1k, Resistor_SMD:R_0402_1005Metric, F.Cu at (82.2, 67.6)
- added R45: 1k, Resistor_SMD:R_0402_1005Metric, F.Cu at (82.2, 69.6)
- added R46: 1k, Resistor_SMD:R_0402_1005Metric, F.Cu at (82.2, 71.6)
- added R47: 1k, Resistor_SMD:R_0402_1005Metric, F.Cu at (82.2, 73.5)
- added R48: 10k, Resistor_SMD:R_0402_1005Metric, F.Cu at (85.1, 61.6)
- added R49: 10k, Resistor_SMD:R_0402_1005Metric, F.Cu at (85.1, 63.6)
- added R50: 10k, Resistor_SMD:R_0402_1005Metric, F.Cu at (85.1, 65.6)
- added R51: 10k, Resistor_SMD:R_0402_1005Metric, F.Cu at (85.1, 67.6)
- added R52: 30k, Resistor_SMD:R_0402_1005Metric, F.Cu at (85.1, 69.6)
- added R53: 1.13k, Resistor_SMD:R_0402_1005Metric, F.Cu at (85.1, 71.6)
- added R54: 1.13k, Resistor_SMD:R_0402_1005Metric, F.Cu at (85.1, 73.5)
- added R55: 1k, Resistor_SMD:R_0402_1005Metric, F.Cu at (88.0, 61.6)
- added R56: 10k, Resistor_SMD:R_0402_1005Metric, F.Cu at (88.0, 63.6)
- added R57: 1k, Resistor_SMD:R_0402_1005Metric, F.Cu at (88.0, 65.6)
- added R58: 10k, Resistor_SMD:R_0402_1005Metric, F.Cu at (88.0, 67.6)
- added SW10: RIGHT_RIGHT, Button_Switch_THT:SW_PUSH-12mm, F.Cu at (217.2, 133.1)
- added SW11: RIGHT_UP, Button_Switch_THT:SW_PUSH-12mm, F.Cu at (198.5, 109.8)
- added SW12: RIGHT_DOWN, Button_Switch_THT:SW_PUSH-12mm, F.Cu at (198.5, 138.8)
- added SW13: RIGHT_LEFT, Button_Switch_THT:SW_PUSH-12mm, F.Cu at (192.2, 120.6)
- added SW14: LEFT_SEL, Button_Switch_THT:SW_PUSH-12mm, F.Cu at (79.2, 123.8)
- added SW15: RIGHT_SEL, Button_Switch_THT:SW_PUSH-12mm, F.Cu at (198.5, 124.3)
- added SW6: LEFT_LEFT, Button_Switch_THT:SW_PUSH-12mm, F.Cu at (68.0, 132.6)
- added SW7: LEFT_RIGHT, Button_Switch_THT:SW_PUSH-12mm, F.Cu at (98.0, 132.6)
- added SW8: LEFT_UP, Button_Switch_THT:SW_PUSH-12mm, F.Cu at (79.2, 109.3)
- added SW9: LEFT_DOWN, Button_Switch_THT:SW_PUSH-12mm, F.Cu at (79.2, 138.3)
- added U11: MPU-6050, Sensor_Motion:InvenSense_QFN-24_4x4mm_P0.5mm, F.Cu at (81.0, 85.6)
- added UD5: BLUE, LED_SMD:LED_0805_2012Metric, F.Cu at (86.4, 83.9)
- added UD6: BLUE, LED_SMD:LED_0805_2012Metric, F.Cu at (86.4, 87.0)
- J5: value USB_C_Receptacle_USB2.0_14P -> Conn_01x14_Pin; footprint Connector_USB:USB_C_Receptacle_G-Switch_GT-USB-7010ASV -> Connector_PinHeader_1.00mm:PinHeader_1x14_P1.00mm_Vertical
- R18, R19: value 5.1k -> 1k; moved to F.Cu
- moved U9 98.9 mm to (143.7, 155.2), turned to -90 degrees
- moved R2 96.7 mm to (145.5, 154.1), turned to -90 degrees
- moved R1 96.7 mm to (141.8, 154.1), turned to -90 degrees
- moved R19 95.0 mm to (79.3, 63.6), turned to 0 degrees
- moved R18 91.8 mm to (79.3, 61.6), turned to 0 degrees
- moved J1 90.3 mm to (144.0, 146.3), turned to 0 degrees
- moved J5 85.5 mm to (163.5, 56.8), turned to 0 degrees
- moved D4 21.2 mm to (157.3, 145.5), turned to 180 degrees
- moved D5 20.5 mm to (157.3, 144.5), turned to 180 degrees
- moved D3 19.7 mm to (157.1, 132.5), turned to 180 degrees
- moved D2 19.0 mm to (157.1, 134.0), turned to 180 degrees
- moved R32 18.9 mm to (155.3, 145.6), turned to 0 degrees
- moved R29 18.8 mm to (157.6, 137.7), turned to 90 degrees
- moved R33 18.1 mm to (155.3, 144.5), turned to 0 degrees
- moved J7 17.7 mm to (151.7, 148.1), turned to -90 degrees
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Connections:
- C1 pad 2: GND -> PGND
- C10 pad 2: GND -> PGND
- C11 pad 2: GND -> PGND
- C12 pad 2: GND -> PGND
- C13 pad 2: GND -> PGND
- C14 pad 2: GND -> PGND
- C15 pad 2: GND -> PGND
- C16 pad 2: GND -> PGND
- C17 pad 2: GND -> PGND
- C18 pad 2: GND -> PGND
- C19 pad 2: GND -> PGND
- C2 pad 2: GND -> PGND
- C20 pad 2: GND -> PGND
- C21 pad 2: GND -> PGND
- C22 pad 2: GND -> PGND
- C23 pad 2: GND -> PGND
- C29 pad 1: +P3V3 -> +3V3
- C3 pad 2: GND -> PGND
- C32 pad 1: +P3V3 -> +3V3
- C33 pad 1: +P3V3 -> +3V3
- C34 pad 1: +P3V3 -> +3V3
- C35 pad 1: +P3V3 -> +3V3
- C36 pad 1: +P3V3 -> +3V3
- C37 pad 1: +P3V3 -> +3V3
- C38 pad 1: +P3V3 -> +3V3
- C39 pad 1: +P3V3 -> +3V3
- C4 pad 2: GND -> PGND
- C40 pad 1: +P3V3 -> +3V3
- C41 pad 1: +P3V3 -> +3V3
- C42 pad 1: +P3V3 -> +3V3
- C5 pad 2: GND -> PGND
- C6 pad 2: GND -> PGND
- C7 pad 2: GND -> PGND
- C8 pad 2: GND -> PGND
- C9 pad 2: GND -> PGND
- J1 pad A1: GND -> PGND
- J1 pad A12: GND -> PGND
- J1 pad B1: GND -> PGND
- J1 pad B12: GND -> PGND
- J1 pad S1: GND -> PGND
- J6 pad 3: GND -> PGND
- PD1 pad 1: GND -> PGND
- PD2 pad 1: GND -> PGND
- R1 pad 2: GND -> PGND
- R18 pad 1: Net-(J5-CC1) -> +3V3
- R18 pad 2: PGND -> Net-(UD5-A)
- R19 pad 1: Net-(J5-CC2) -> +3V3
- R19 pad 2: PGND -> Net-(UD6-A)
- R2 pad 2: GND -> PGND
- R34 pad 1: GND -> PGND
- R35 pad 1: GND -> PGND
- R4 pad 2: GND -> PGND
- SW1 pad 1: GND -> PGND
- U1 pad 4: GND -> PGND
- U2 pad 1: GND -> PGND
- U3 pad 62: GND -> PGND
- U3 pad 66: Net-(U3-USB_DM) -> unconnected-(U3-USB_DM-Pad66)
- U3 pad 67: Net-(U3-USB_DP) -> unconnected-(U3-USB_DP-Pad67)
- U3 pad 81: GND -> PGND
- U4 pad 8: +P3V3 -> +3V3
- U6 pad 1: +P3V3 -> +3V3
- U6 pad 10: +P3V3 -> +3V3
- U6 pad 22: +P3V3 -> +3V3
- U6 pad 33: +P3V3 -> +3V3
- U6 pad 42: +P3V3 -> +3V3
- U6 pad 43: +P3V3 -> +3V3
- U6 pad 44: +P3V3 -> +3V3
- U6 pad 48: +P3V3 -> +3V3
- U6 pad 49: +P3V3 -> +3V3
- U7 pad 5: +P3V3 -> +3V3
- U8 pad 5: +P3V3 -> +3V3
- U9 pad 2: GND -> PGND
- Y1 pad 2: GND -> PGND
- Y1 pad 4: GND -> PGND
Routing:
- net GND: track 80.1 -> 0.00 mm, vias 16 -> 0
- net +3V3: track 170.0 -> 235.9 mm, vias 11 -> 17
- net +P3V3: track 65.9 -> 0.00 mm, vias 6 -> 0
- net PGND: track 60.4 -> 111.2 mm, vias 9 -> 23
- net /USB_D-: track 40.5 -> 0.00 mm, vias 2 -> 0
- net /USB_D+: track 40.4 -> 0.00 mm, vias 2 -> 0
- net /GPIO24: track 41.1 -> 2.82 mm, vias 2 -> 1
- net /GPIO23: track 34.7 -> 3.00 mm, vias 2 -> 1
- net /GPIO25: track 31.0 -> 0.00 mm, vias 2 -> 0
- net /GPIO47_ADC7: track 30.2 -> 0.00 mm
- net /GPIO46_ADC6: track 28.3 -> 0.93 mm
- net (no net): track 0.00 -> 26.5 mm, vias 0 -> 3
- net P_VBUS: track 26.5 -> 0.00 mm, vias 3 -> 0
- net /GPIO1: track 26.4 -> 0.00 mm, vias 1 -> 0
- net /GPIO45_ADC5: track 26.7 -> 0.73 mm
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- removed copper zone on F.Cu, net (none)
- removed copper zone on In1.Cu, net (none)
- removed copper zone on In2.Cu, net (none)
- removed copper zone on B.Cu, net GND
- removed copper zone on B.Cu, net PGND
Other:
- board size 20.3 x 99.1 mm -> 25.6 x 96.1 mm
- board text removed: "0"
- board text removed: "1"
- board text removed: "10"
- board text removed: "11"
- board text removed: "12"
- board text removed: "13"
- board text removed: "14"
- board text removed: "15"
- board text removed: "16"
- board text removed: "17"
- board text removed: "18"
- board text removed: "19"
- board text removed: "2"
- board text removed: "20"
- board text removed: "27"
- board text removed: "28"
- board text removed: "29"
- board text removed: "3"
- board text removed: "30"
- board text removed: "31"
- board text removed: "32"
- board text removed: "33"
- board text removed: "34"
- board text removed: "35"
- board text removed: "36"
- board text removed: "37"
- board text removed: "38"
- board text removed: "39"
- board text removed: "4"
- board text removed: "40"
- board text removed: "41"
- board text removed: "42"
- board text removed: "43"
- board text removed: "44"
- board text removed: "45"
- board text removed: "46"
- board text removed: "47"
- board text removed: "5"
- board text removed: "6"
- board text removed: "7"
- board text removed: "8"
- board text removed: "9"
